File: KiCad/Numpadulator.sch (KiCad schematic (older format))
At the start: 58 parts, among them SW1 Cherry_MX_RGB_WS2812, SW10 Cherry_MX_RGB_WS2812, SW11 Cherry_MX_RGB_WS2812, SW12 Cherry_MX_RGB_WS2812, SW13 Cherry_MX_RGB_WS2812, SW14 Cherry_MX_RGB_WS2812, SW15 Cherry_MX_RGB_WS2812, SW16 Cherry_MX_RGB_WS2812, SW17 Cherry_MX_RGB_WS2812, SW18 Cherry_MX_RGB_WS2812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

Commit message: Started fleshing out pcb, need to change large keys
Parts:
- C1, C10, C11, C12, C13, C14, C15, C16, C17, C18, C2, C3, C4, C5, C6, C7, C8, C9: footprint (none) -> Capacitor_SMD:C_0805_2012Metric
- D1, D10, D11, D12, D13, D14, D15, D16, D17, D18, D19, D2, D3, D4, D5, D6, D7, D8, D9: footprint (none) -> Diode_SMD:D_SOD-123
- SW1, SW10, SW11, SW12, SW13, SW14, SW15, SW16, SW17, SW18, SW2, SW3, SW4, SW5, SW6, SW7, SW8, SW9: footprint (none) -> Cherry MX:Cherry-MX_PCB-Mounted_LTST-A683CEGBW_Kailh_Socket
- SW19: footprint (none) -> Custom-parts:XDCR_PEC11R-4215F-S0024
- U2: footprint (none) -> Display:Adafruit_SSD1306

Commit message: More layout and frustration 3:
Parts:
- removed SW17, SW18, SW6: Cherry_MX_RGB_WS2812, Cherry MX:Cherry-MX_PCB-Mounted_LTST-A683CEGBW_Kailh_Socket, symbol Custom_Library:Cherry_MX_RGB_WS2812
- added D20, D21, D22: WS2816, Custom-parts:SK6812-MINI-E, symbol Cherry_MX:WS2816
- added MX1, MX2, MX3: MX-NoLED, MX_Only:MXOnly-2U-Hotswap, symbol MX_Alps_Hybrid:MX-NoLED
- SW1, SW10, SW11, SW12, SW13, SW14, SW15, SW16, SW2, SW3, SW4, SW5, SW7, SW8, SW9: footprint Cherry MX:Cherry-MX_PCB-Mounted_LTST-A683CEGBW_Kailh_Socket -> Custom-parts:Cherry-MX_PCB-Mounted_SK6812-MINI-E_Kailh_Socket
Connections:
- net COL0: now also MX1.1 (COL)
- net COL3: now also MX2.1 (COL), MX3.1 (COL)
- net GND: now also D20.3 (GND), D21.3 (GND), D22.3 (GND)
- net VCC: now also D20.1 (VCC), D21.1 (VCC), D22.1 (VCC)
- net at SW12.2 (DOUT): now also D21.4 (DIN)
- net at SW4.4 (DIN): now also D21.2 (DOUT)
- net at D17.2 (A): now also MX2.2 (ROW)
- net at SW14.2 (DOUT): now also D22.4 (DIN)
- net at D18.2 (A): now also MX3.2 (ROW)
- net at D6.2 (A): now also MX1.2 (ROW)
- net at SW15.4 (DIN): now also D20.2 (DOUT)
- new net: D20.4 (DIN), D22.2 (DOUT)
Changed lines of the file:
@@
 F 0 "SW7" H 3200 2825 50  0000 C CNN
 F 1 "Cherry_MX_RGB_WS2812" H 3200 2734 50  0000 C CNN
-F 2 "Cherry MX:Cherry-MX_PCB-Mounted_LTST-A683CEGBW_Kailh_Socket" H 3200 2350 50  0001 C CNN
+F 2 "Custom-parts:Cherry-MX_PCB-Mounted_SK6812-MINI-E_Kailh_Socket" H 3200 2350 50  0001 C CNN
 F 3 "" H 3200 2350 50  0001 C CNN
 	1    3200 2350
@@
 F 0 "SW2" H 1525 2825 50  0000 C CNN
 F 1 "Cherry_MX_RGB_WS2812" H 1525 2734 50  0000 C CNN
-F 2 "Cherry MX:Cherry-MX_PCB-Mounted_LTST-A683CEGBW_Kailh_Socket" H 1525 2350 50  0001 C CNN
+F 2 "Custom-parts:Cherry-MX_PCB-Mounted_SK6812-MINI-E_Kailh_Socket" H 1525 2350 50  0001 C CNN
 F 3 "" H 1525 2350 50  0001 C CNN
 	1    1525 2350
@@
 F 0 "SW1" H 1525 1900 50  0000 C CNN
 F 1 "Cherry_MX_RGB_WS2812" H 1525 1809 50  0000 C CNN
-F 2 "Cherry MX:Cherry-MX_PCB-Mounted_LTST-A683CEGBW_Kailh_Socket" H 1525 1425 50  0001 C CNN
+F 2 "Custom-parts:Cherry-MX_PCB-Mounted_SK6812-MINI-E_Kailh_Socket" H 1525 1425 50  0001 C CNN
 F 3 "" H 1525 1425 50  0001 C CNN
 	1    1525 1425
@@
 F 0 "SW11" H 4875 2825 50  0000 C CNN
 F 1 "Cherry_MX_RGB_WS2812" H 4875 2734 50  0000 C CNN
-F 2 "Cherry MX:Cherry-MX_PCB-Mounted_LTST-A683CEGBW_Kailh_Socket" H 4875 2350 50  0001 C CNN
+F 2 "Custom-parts:Cherry-MX_PCB-Mounted_SK6812-MINI-E_Kailh_Socket" H 4875 2350 50  0001 C CNN
 F 3 "" H 4875 2350 50  0001 C CNN
 	1    4875 2350
@@
 F 0 "SW16" H 6550 2825 50  0000 C CNN
 F 1 "Cherry_MX_RGB_WS2812" H 6550 2734 50  0000 C CNN
-F 2 "Cherry MX:Cherry-MX_PCB-Mounted_LTST-A683CEGBW_Kailh_Socket" H 6550 2350 50  0001 C CNN
+F 2 "Custom-parts:Cherry-MX_PCB-Mounted_SK6812-MINI-E_Kailh_Socket" H 6550 2350 50  0001 C CNN
 F 3 "" H 6550 2350 50  0001 C CNN
 	1    6550 2350
@@
 F 0 "SW8" H 3200 3825 50  0000 C CNN
 F 1 "Cherry_MX_RGB_WS2812" H 3200 3734 50  0000 C CNN
-F 2 "Cherry MX:Cherry-MX_PCB-Mounted_LTST-A683CEGBW_Kailh_Socket" H 3200 3350 50  0001 C CNN
+F 2 "Custom-parts:Cherry-MX_PCB-Mounted_SK6812-MINI-E_Kailh_Socket" H 3200 3350 50  0001 C CNN
 F 3 "" H 3200 3350 50  0001 C CNN
 	1    3200 3350
@@
 F 0 "SW3" H 1525 3825 50  0000 C CNN
 F 1 "Cherry_MX_RGB_WS2812" H 1525 3734 50  0000 C CNN
-F 2 "Cherry MX:Cherry-MX_PCB-Mounted_LTST-A683CEGBW_Kailh_Socket" H 1525 3350 50  0001 C CNN
+F 2 "Custom-parts:Cherry-MX_PCB-Mounted_SK6812-MINI-E_Kailh_Socket" H 1525 3350 50  0001 C CNN
 F 3 "" H 1525 3350 50  0001 C CNN
 	1    1525 3350
@@
 F 0 "SW12" H 4875 3825 50  0000 C CNN
 F 1 "Cherry_MX_RGB_WS2812" H 4875 3734 50  0000 C CNN
-F 2 "Cherry MX:Cherry-MX_PCB-Mounted_LTST-A683CEGBW_Kailh_Socket" H 4875 3350 50  0001 C CNN
+F 2 "Custom-parts:Cherry-MX_PCB-Mounted_SK6812-MINI-E_Kailh_Socket" H 4875 3350 50  0001 C CNN
 F 3 "" H 4875 3350 50  0001 C CNN
 	1    4875 3350
@@
 Wire Wire Line
 	5550 3300 5550 3400
-Wire Wire Line
-	5550 3400 6225 3400
-Wire Wire Line
-	6875 3200 7125 3200
-Wire Wire Line
-	6875 3100 7075 3100
-$Comp
-L Custom_Library:Cherry_MX_RGB_WS2812 SW17
-U 1 1 5F2E4652
-P 6550 3350
-F 0 "SW17" H 6550 3825 50  0000 C CNN
-F 1 "Cherry_MX_RGB_WS2812" H 6550 3734 50  0000 C CNN
-F 2 "Cherry MX:Cherry-MX_PCB-Mounted_LTST-A683CEGBW_Kailh_Socket" H 6550 3350 50  0001 C CNN
-F 3 "" H 6550 3350 50  0001 C CNN
-	1    6550 3350
-	1    0    0    -1
-$EndComp
-Wire Wire Line
-	6875 3300 7225 3300
 $Comp
 L Device:C_Small C17
 U 1 1 5F2E4659
 P 5975 3050
-F 0 "C17" H 5800 3000 50  0000 L CNN
+F 0 "C17" H 5800 2975 50  0000 L CNN
 F 1 "0.1uF" H 5725 3125 50  0000 L CNN
 F 2 "Capacitor_SMD:C_0805_2012Metric" H 5975 3050 50  0001 C CNN
@@
 Wire Wire Line
 	2300 1600 7350 1600
-Wire Wire Line
-	7075 2100 7075 3100
 Connection ~ 7075 2100
 Wire Wire Line
@@
 F 0 "SW9" H 3200 4825 50  0000 C CNN
 F 1 "Cherry_MX_RGB_WS2812" H 3200 4734 50  0000 C CNN
-F 2 "Cherry MX:Cherry-MX_PCB-Mounted_LTST-A683CEGBW_Kailh_Socket" H 3200 4350 50  0001 C CNN
+F 2 "Custom-parts:Cherry-MX_PCB-Mounted_SK6812-MINI-E_Kailh_Socket" H 3200 4350 50  0001 C CNN
 F 3 "" H 3200 4350 50  0001 C CNN
 	1    3200 4350
@@
 F 0 "SW4" H 1525 4825 50  0000 C CNN
 F 1 "Cherry_MX_RGB_WS2812" H 1525 4734 50  0000 C CNN
-F 2 "Cherry MX:Cherry-MX_PCB-Mounted_LTST-A683CEGBW_Kailh_Socket" H 1525 4350 50  0001 C CNN
+F 2 "Custom-parts:Cherry-MX_PCB-Mounted_SK6812-MINI-E_Kailh_Socket" H 1525 4350 50  0001 C CNN
 F 3 "" H 1525 4350 50  0001 C CNN
 	1    1525 4350
@@
 F 0 "SW13" H 4875 4825 50  0000 C CNN
 F 1 "Cherry_MX_RGB_WS2812" H 4875 4734 50  0000 C CNN
-F 2 "Cherry MX:Cherry-MX_PCB-Mounted_LTST-A683CEGBW_Kailh_Socket" H 4875 4350 50  0001 C CNN
+F 2 "Custom-parts:Cherry-MX_PCB-Mounted_SK6812-MINI-E_Kailh_Socket" H 4875 4350 50  0001 C CNN
 F 3 "" H 4875 4350 50  0001 C CNN
 	1    4875 4350
@@
 F 0 "SW10" H 3200 5825 50  0000 C CNN
 F 1 "Cherry_MX_RGB_WS2812" H 3200 5734 50  0000 C CNN
-F 2 "Cherry MX:Cherry-MX_PCB-Mounted_LTST-A683CEGBW_Kailh_Socket" H 3200 5350 50  0001 C CNN
+F 2 "Custom-parts:Cherry-MX_PCB-Mounted_SK6812-MINI-E_Kailh_Socket" H 3200 5350 50  0001 C CNN
 F 3 "" H 3200 5350 50  0001 C CNN
 	1    3200 5350
@@
 F 0 "SW5" H 1525 5825 50  0000 C CNN
 F 1 "Cherry_MX_RGB_WS2812" H 1525 5734 50  0000 C CNN
-F 2 "Cherry MX:Cherry-MX_PCB-Mounted_LTST-A683CEGBW_Kailh_Socket" H 1525 5350 50  0001 C CNN
+F 2 "Custom-parts:Cherry-MX_PCB-Mounted_SK6812-MINI-E_Kailh_Socket" H 1525 5350 50  0001 C CNN
 F 3 "" H 1525 5350 50  0001 C CNN
 	1    1525 5350
@@
 F 0 "SW14" H 4875 5825 50  0000 C CNN
 F 1 "Cherry_MX_RGB_WS2812" H 4875 5734 50  0000 C CNN
-F 2 "Cherry MX:Cherry-MX_PCB-Mounted_LTST-A683CEGBW_Kailh_Socket" H 4875 5350 50  0001 C CNN
+F 2 "Custom-parts:Cherry-MX_PCB-Mounted_SK6812-MINI-E_Kailh_Socket" H 4875 5350 50  0001 C CNN
 F 3 "" H 4875 5350 50  0001 C CNN
 	1    4875 5350
@@
 Wire Wire Line
 	5550 5400 6225 5400
-Wire Wire Line
-	6875 5200 7125 5200
-Wire Wire Line
-	6875 5100 7075 5100
-$Comp
-L Custom_Library:Cherry_MX_RGB_WS2812 SW18
-U 1 1 5F4DF220
-P 6550 5350
-F 0 "SW18" H 6550 5825 50  0000 C CNN
-F 1 "Cherry_MX_RGB_WS2812" H 6550 5734 50  0000 C CNN
-F 2 "Cherry MX:Cherry-MX_PCB-Mounted_LTST-A683CEGBW_Kailh_Socket" H 6550 5350 50  0001 C CNN
-F 3 "" H 6550 5350 50  0001 C CNN
-	1    6550 5350
-	1    0    0    -1
-$EndComp
-Wire Wire Line
-	6875 5300 7225 5300
 $Comp
 L Device:C_Small C18
@@
 $EndComp
 Wire Wire Line
-	2050 5100 2050 6100
+	2050 5100 2050 6000
 Wire Wire Line
 	5400 5100 5400 6100
@@
 Connection ~ 5400 4100
 Wire Wire Line
-	7075 3100 7075 5100
-Connection ~ 7075 3100
-Wire Wire Line
 	5550 4625 1075 4625
 Wire Wire Line
@@
 Wire Wire Line
 	2300 6200 2300 6525
-Wire Wire Line
-	1850 6200 2100 6200
 $Comp
 L Device:D_Small D6
@@
 	-1   0    0    1
 $EndComp
-Wire Wire Line
-	1850 6100 2050 6100
-$Comp
-L Custom_Library:Cherry_MX_RGB_WS2812 SW6
-U 1 1 5F560ACB
-P 1525 6350
-F 0 "SW6" H 1525 6825 50  0000 C CNN
-F 1 "Cherry_MX_RGB_WS2812" H 1525 6734 50  0000 C CNN
-F 2 "Cherry MX:Cherry-MX_PCB-Mounted_LTST-A683CEGBW_Kailh_Socket" H 1525 6350 50  0001 C CNN
-F 3 "" H 1525 6350 50  0001 C CNN
-	1    1525 6350
-	1    0    0    -1
-$EndComp
 $Comp
 L Device:C_Small C5
@@
 Wire Wire Line
 	1075 6400 1200 6400
-Wire Wire Line
-	1850 6300 2200 6300
 Wire Wire Line
 	2200 6300 2200 6400
@@
 F 0 "SW15" H 4875 6825 50  0000 C CNN
 F 1 "Cherry_MX_RGB_WS2812" H 4875 6734 50  0000 C CNN
-F 2 "Cherry MX:Cherry-MX_PCB-Mounted_LTST-A683CEGBW_Kailh_Socket" H 4875 6350 50  0001 C CNN
+F 2 "Custom-parts:Cherry-MX_PCB-Mounted_SK6812-MINI-E_Kailh_Socket" H 4875 6350 50  0001 C CNN
 F 3 "" H 4875 6350 50  0001 C CNN
 	1    4875 6350
@@
 NoConn ~ 9200 975
 NoConn ~ 10200 875
+$Comp
+L MX_Alps_Hybrid:MX-NoLED MX2
+U 1 1 5F27E9E0
+P 6925 3050
+F 0 "MX2" H 6958 3273 60  0000 C CNN
+F 1 "MX-NoLED" H 6958 3199 20  0000 C CNN
+F 2 "MX_Only:MXOnly-2U-Hotswap" H 6300 3025 60  0001 C CNN
+F 3 "" H 6300 3025 60  0001 C CNN
+	1    6925 3050
+	1    0    0    -1
+$EndComp
+$Comp
+L MX_Alps_Hybrid:MX-NoLED MX3
+U 1 1 5F2924E7
+P 6925 5050
+F 0 "MX3" H 6958 5273 60  0000 C CNN
+F 1 "MX-NoLED" H 6958 5199 20  0000 C CNN
+F 2 "MX_Only:MXOnly-2U-Hotswap" H 6300 5025 60  0001 C CNN
+F 3 "" H 6300 5025 60  0001 C CNN
+	1    6925 5050
+	1    0    0    -1
+$EndComp
+$Comp
+L MX_Alps_Hybrid:MX-NoLED MX1
+U 1 1 5F2A7123
+P 1900 6050
+F 0 "MX1" H 1933 6273 60  0000 C CNN
+F 1 "MX-NoLED" H 1933 6199 20  0000 C CNN
+F 2 "MX_Only:MXOnly-2U-Hotswap" H 1275 6025 60  0001 C CNN
+F 3 "" H 1275 6025 60  0001 C CNN
+	1    1900 6050
+	1    0    0    -1
+$EndComp
+$Comp
+L Cherry_MX:WS2816 D21
+U 1 1 5F2BB67C
+P 6550 3350
+F 0 "D21" H 6550 3625 50  0000 C CNN
+F 1 "WS2816" H 6550 3534 50  0000 C CNN
+F 2 "Custom-parts:SK6812-MINI-E" H 6425 3350 50  0001 C CNN
+F 3 "" H 6425 3350 50  0001 C CNN
+	1    6550 3350
+	1    0    0    -1
+$EndComp
+Wire Wire Line
+	7075 2100 7075 3000
+Connection ~ 7075 3000
+Wire Wire Line
+	7075 3000 7075 5000
+Wire Wire Line
+	6875 3200 7125 3200
+Wire Wire Line
+	5550 3400 6225 3400
+Wire Wire Line
+	6875 3300 7225 3300
+Wire Wire Line
+	6875 5200 7125 5200
+$Comp
+L Cherry_MX:WS2816 D22
+U 1 1 5F415D00
+P 6550 5350
+F 0 "D22" H 6550 5625 50  0000 C CNN
+F 1 "WS2816" H 6550 5534 50  0000 C CNN
+F 2 "Custom-parts:SK6812-MINI-E" H 6425 5350 50  0001 C CNN
+F 3 "" H 6425 5350 50  0001 C CNN
+	1    6550 5350
+	1    0    0    -1
+$EndComp
+Wire Wire Line
+	6875 5300 7225 5300
+Wire Wire Line
+	1850 6200 2100 6200
+$Comp
+L Cherry_MX:WS2816 D20
+U 1 1 5F4E82F7
+P 1525 6350
+F 0 "D20" H 1525 6625 50  0000 C CNN
+F 1 "WS2816" H 1525 6534 50  0000 C CNN
+F 2 "Custom-parts:SK6812-MINI-E" H 1400 6350 50  0001 C CNN
+F 3 "" H 1400 6350 50  0001 C CNN
+	1    1525 6350
+	1    0    0    -1
+$EndComp
+Wire Wire Line
+	1850 6300 2200 6300
 $EndSCHEMATC

Commit message: Moved MCU via the Genius of WIll
Parts:
- C1, C10, C11, C12, C13, C14, C15, C16, C17, C18, C2, C3, C4, C5, C6, C7, C8, C9: symbol Device:C_Small -> Numpadulator-rescue:C_Small-Device
- D1, D10, D11, D12, D13, D14, D15, D16, D17, D18, D19, D2, D3, D4, D5, D6, D7, D8, D9: symbol Device:D_Small -> Numpadulator-rescue:D_Small-Device
- SW19: symbol Device:Rotary_Encoder_Switch -> Numpadulator-rescue:Rotary_Encoder_Switch-Device
