File: KiCad/Numpadulator.sch (KiCad schematic (older format))
At the start: 74 parts, among them SW1 Cherry_MX_RGB_WS2812, SW10 Cherry_MX_RGB_WS2812, SW11 Cherry_MX_RGB_WS2812, SW12 Cherry_MX_RGB_WS2812, SW13 Cherry_MX_RGB_WS2812, SW14 Cherry_MX_RGB_WS2812, SW15 Cherry_MX_RGB_WS2812, SW16 Cherry_MX_RGB_WS2812, SW19 Rotary_Encoder_Switch, SW2 Cherry_MX_RGB_WS2812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

Commit message: forgot to save
Parts:
- gave numbers to parts that had none: 6
Changed lines of the file:
@@
 $EndComp
 $Comp
-L Numpadulator-rescue:C_Small-Device C?
+L Numpadulator-rescue:C_Small-Device C21
 U 1 1 6036FCAA
 P 2575 850
-F 0 "C?" H 2425 900 50  0000 L CNN
+F 0 "C21" H 2425 900 50  0000 L CNN
 F 1 "0.1uF" H 2300 825 50  0000 L CNN
 F 2 "Capacitor_SMD:C_0805_2012Metric" H 2575 850 50  0001 C CNN
@@
 $EndComp
 $Comp
-L Numpadulator-rescue:GND-power #PWR?
+L Numpadulator-rescue:GND-power #PWR0161
 U 1 1 6036FCB0
 P 2475 850
-F 0 "#PWR?" H 2475 600 50  0001 C CNN
+F 0 "#PWR0161" H 2475 600 50  0001 C CNN
 F 1 "GND" H 2480 677 50  0000 C CNN
 F 2 "" H 2475 850 50  0001 C CNN
@@
 Connection ~ 2875 850
 $Comp
-L power:VCC #PWR?
+L power:VCC #PWR0162
 U 1 1 603D37AD
 P 2875 725
-F 0 "#PWR?" H 2875 575 50  0001 C CNN
+F 0 "#PWR0162" H 2875 575 50  0001 C CNN
 F 1 "VCC" H 2890 898 50  0000 C CNN
 F 2 "" H 2875 725 50  0001 C CNN
@@
 $EndComp
 $Comp
-L power:GND #PWR?
+L power:GND #PWR0163
 U 1 1 603E8BB9
 P 2875 1525
-F 0 "#PWR?" H 2875 1275 50  0001 C CNN
+F 0 "#PWR0163" H 2875 1275 50  0001 C CNN
 F 1 "GND" V 2880 1397 50  0000 R CNN
 F 2 "" H 2875 1525 50  0001 C CNN
@@
 $EndComp
 $Comp
-L Numpadulator-rescue:C_Small-Device C?
+L Numpadulator-rescue:C_Small-Device C22
 U 1 1 603EC8B5
 P 4250 850
-F 0 "C?" H 4100 900 50  0000 L CNN
+F 0 "C22" H 4100 900 50  0000 L CNN
 F 1 "0.1uF" H 3975 825 50  0000 L CNN
 F 2 "Capacitor_SMD:C_0805_2012Metric" H 4250 850 50  0001 C CNN
@@
 $EndComp
 $Comp
-L Numpadulator-rescue:GND-power #PWR?
+L Numpadulator-rescue:GND-power #PWR0164
 U 1 1 603EC8BB
 P 4150 850
-F 0 "#PWR?" H 4150 600 50  0001 C CNN
+F 0 "#PWR0164" H 4150 600 50  0001 C CNN
 F 1 "GND" H 4155 677 50  0000 C CNN
 F 2 "" H 4150 850 50  0001 C CNN
@@
 Connection ~ 4550 850
 $Comp
-L power:VCC #PWR?
+L power:VCC #PWR0165
 U 1 1 603EC8C5
 P 4550 725
-F 0 "#PWR?" H 4550 575 50  0001 C CNN
+F 0 "#PWR0165" H 4550 575 50  0001 C CNN
 F 1 "VCC" H 4565 898 50  0000 C CNN
 F 2 "" H 4550 725 50  0001 C CNN
@@
 	3175 1225 4250 1225
 $Comp
-L power:GND #PWR?
+L power:GND #PWR0166
 U 1 1 60462919
 P 4550 1525
-F 0 "#PWR?" H 4550 1275 50  0001 C CNN
+F 0 "#PWR0166" H 4550 1275 50  0001 C CNN
 F 1 "GND" V 4555 1397 50  0000 R CNN
 F 2 "" H 4550 1525 50  0001 C CNN
@@
 	2875 3500 2875 3400
 $Comp
-L Numpadulator-rescue:C_Small-Device C?
+L Numpadulator-rescue:C_Small-Device C19
 U 1 1 60565279
 P -275 2875
-F 0 "C?" H -425 2925 50  0000 L CNN
+F 0 "C19" H -425 2925 50  0000 L CNN
 F 1 "0.1uF" H -550 2850 50  0000 L CNN
 F 2 "Capacitor_SMD:C_0805_2012Metric" H -275 2875 50  0001 C CNN
@@
 $EndComp
 $Comp
-L Numpadulator-rescue:GND-power #PWR?
+L Numpadulator-rescue:GND-power #PWR0167
 U 1 1 6056527F
 P -375 2875
-F 0 "#PWR?" H -375 2625 50  0001 C CNN
+F 0 "#PWR0167" H -375 2625 50  0001 C CNN
 F 1 "GND" H -370 2702 50  0000 C CNN
 F 2 "" H -375 2875 50  0001 C CNN
@@
 Connection ~ 25   2875
 $Comp
-L power:VCC #PWR?
+L power:VCC #PWR0168
 U 1 1 60565289
 P 25 2750
-F 0 "#PWR?" H 25  2600 50  0001 C CNN
+F 0 "#PWR0168" H 25  2600 50  0001 C CNN
 F 1 "VCC" H 40  2923 50  0000 C CNN
 F 2 "" H 25  2750 50  0001 C CNN
@@
 $EndComp
 $Comp
-L power:GND #PWR?
+L power:GND #PWR0169
 U 1 1 60579C82
 P 25 3550
-F 0 "#PWR?" H 25  3300 50  0001 C CNN
+F 0 "#PWR0169" H 25  3300 50  0001 C CNN
 F 1 "GND" H 30  3377 50  0000 C CNN
 F 2 "" H 25  3550 50  0001 C CNN
@@
 Connection ~ 8125 3300
 $Comp
-L Numpadulator-rescue:C_Small-Device C?
+L Numpadulator-rescue:C_Small-Device C24
 U 1 1 605D42B2
 P 7525 2925
-F 0 "C?" H 7375 2975 50  0000 L CNN
+F 0 "C24" H 7375 2975 50  0000 L CNN
 F 1 "0.1uF" H 7250 2900 50  0000 L CNN
 F 2 "Capacitor_SMD:C_0805_2012Metric" H 7525 2925 50  0001 C CNN
@@
 $EndComp
 $Comp
-L Numpadulator-rescue:GND-power #PWR?
+L Numpadulator-rescue:GND-power #PWR0170
 U 1 1 605D42B8
 P 7425 2925
-F 0 "#PWR?" H 7425 2675 50  0001 C CNN
+F 0 "#PWR0170" H 7425 2675 50  0001 C CNN
 F 1 "GND" H 7430 2752 50  0000 C CNN
 F 2 "" H 7425 2925 50  0001 C CNN
@@
 Connection ~ 7825 2925
 $Comp
-L power:VCC #PWR?
+L power:VCC #PWR0171
 U 1 1 605D42C2
 P 7825 2800
-F 0 "#PWR?" H 7825 2650 50  0001 C CNN
+F 0 "#PWR0171" H 7825 2650 50  0001 C CNN
 F 1 "VCC" H 7840 2973 50  0000 C CNN
 F 2 "" H 7825 2800 50  0001 C CNN
@@
 $EndComp
 $Comp
-L power:GND #PWR?
+L power:GND #PWR0172
 U 1 1 605E92E4
 P 7825 3600
-F 0 "#PWR?" H 7825 3350 50  0001 C CNN
+F 0 "#PWR0172" H 7825 3350 50  0001 C CNN
 F 1 "GND" H 7830 3427 50  0000 C CNN
 F 2 "" H 7825 3600 50  0001 C CNN
@@
 	550  6400 1200 6400
 $Comp
-L Numpadulator-rescue:C_Small-Device C?
+L Numpadulator-rescue:C_Small-Device C20
 U 1 1 6065A1B9
 P -50 6025
-F 0 "C?" H -200 6075 50  0000 L CNN
+F 0 "C20" H -200 6075 50  0000 L CNN
 F 1 "0.1uF" H -325 6000 50  0000 L CNN
 F 2 "Capacitor_SMD:C_0805_2012Metric" H -50 6025 50  0001 C CNN
@@
 $EndComp
 $Comp
-L Numpadulator-rescue:GND-power #PWR?
+L Numpadulator-rescue:GND-power #PWR0173
 U 1 1 6065A1BF
 P -150 6025
-F 0 "#PWR?" H -150 5775 50  0001 C CNN
+F 0 "#PWR0173" H -150 5775 50  0001 C CNN
 F 1 "GND" H -145 5852 50  0000 C CNN
 F 2 "" H -150 6025 50  0001 C CNN
@@
 Connection ~ 250  6025
 $Comp
-L power:VCC #PWR?
+L power:VCC #PWR0174
 U 1 1 6065A1C9
 P 250 5900
-F 0 "#PWR?" H 250 5750 50  0001 C CNN
+F 0 "#PWR0174" H 250 5750 50  0001 C CNN
 F 1 "VCC" H 265 6073 50  0000 C CNN
 F 2 "" H 250 5900 50  0001 C CNN
@@
 	-425 5625 7225 5625
 $Comp
-L power:GND #PWR?
+L power:GND #PWR0175
 U 1 1 606873EB
 P 250 6700
-F 0 "#PWR?" H 250 6450 50  0001 C CNN
+F 0 "#PWR0175" H 250 6450 50  0001 C CNN
 F 1 "GND" H 255 6527 50  0000 C CNN
 F 2 "" H 250 6700 50  0001 C CNN
@@
 	5200 6300 5750 6300
 $Comp
-L Numpadulator-rescue:C_Small-Device C?
+L Numpadulator-rescue:C_Small-Device C23
 U 1 1 606BA221
 P 5750 5925
-F 0 "C?" H 5600 5975 50  0000 L CNN
+F 0 "C23" H 5600 5975 50  0000 L CNN
 F 1 "0.1uF" H 5475 5900 50  0000 L CNN
 F 2 "Capacitor_SMD:C_0805_2012Metric" H 5750 5925 50  0001 C CNN
@@
 $EndComp
 $Comp
-L Numpadulator-rescue:GND-power #PWR?
+L Numpadulator-rescue:GND-power #PWR0176
 U 1 1 606BA227
 P 5650 5925
-F 0 "#PWR?" H 5650 5675 50  0001 C CNN
+F 0 "#PWR0176" H 5650 5675 50  0001 C CNN
 F 1 "GND" H 5655 5752 50  0000 C CNN
 F 2 "" H 5650 5925 50  0001 C CNN
@@
 Connection ~ 6050 5925
 $Comp
-L power:VCC #PWR?
+L power:VCC #PWR0177
 U 1 1 606BA231
 P 6050 5800
-F 0 "#PWR?" H 6050 5650 50  0001 C CNN
+F 0 "#PWR0177" H 6050 5650 50  0001 C CNN
 F 1 "VCC" H 6065 5973 50  0000 C CNN
 F 2 "" H 6050 5800 50  0001 C CNN
@@
 $EndComp
 $Comp
-L power:GND #PWR?
+L power:GND #PWR0178
 U 1 1 606D0833
 P 6050 6600
-F 0 "#PWR?" H 6050 6350 50  0001 C CNN
+F 0 "#PWR0178" H 6050 6350 50  0001 C CNN
 F 1 "GND" H 6055 6427 50  0000 C CNN
 F 2 "" H 6050 6600 50  0001 C CNN

Commit message: PLACED EVERYTHING I THINK
Connections:
- net at D21.2 (DOUT), D26.3 (DIN): no longer D26.1 (DOUT), SW4.4 (DIN)
- new net: D26.1 (DOUT), SW4.4 (DIN)
Changed lines of the file:
@@
-$EndComp
-$Comp
-L LED:SK6812MINI D26
-U 1 1 6034FC1B
-P 7825 3300
-F 0 "D26" H 8169 3346 50  0000 L CNN
-F 1 "SK6812MINI" H 8169 3255 50  0000 L CNN
-F 2 "LED_SMD:LED_SK6812MINI_PLCC4_3.5x3.5mm_P1.75mm" H 7875 3000 50  0001 L TNN
-F 3 "https://cdn-shop.adafruit.com/product-files/2686/SK6812MINI_REV.01-1-2.pdf" H 7925 2925 50  0001 L TNN
-	1    7825 3300
-	1    0    0    -1
 $EndComp
 $Comp
@@
 $EndComp
 Wire Wire Line
-	7525 3300 8125 3300
-Wire Wire Line
-	6875 3300 7525 3300
-Connection ~ 7525 3300
-Wire Wire Line
 	8125 3300 8125 3625
 Wire Wire Line
 	1075 3625 8125 3625
-Connection ~ 8125 3300
 $Comp
 L Numpadulator-rescue:C_Small-Device C24
@@
 $EndComp
 NoConn ~ 6350 6300
+Wire Wire Line
+	6875 3300 7525 3300
+$Comp
+L LED:SK6812MINI D26
+U 1 1 6034FC1B
+P 7825 3300
+F 0 "D26" H 8169 3346 50  0000 L CNN
+F 1 "SK6812MINI" H 8169 3255 50  0000 L CNN
+F 2 "LED_SMD:LED_SK6812MINI_PLCC4_3.5x3.5mm_P1.75mm" H 7875 3000 50  0001 L TNN
+F 3 "https://cdn-shop.adafruit.com/product-files/2686/SK6812MINI_REV.01-1-2.pdf" H 7925 2925 50  0001 L TNN
+	1    7825 3300
+	1    0    0    -1
+$EndComp
 $EndSCHEMATC
