File: KiCad/Numpadulator.kicad_pcb (KiCad board)
At the start: 2 copper layers, 82.6 x 138.4 mm, 61 parts, among them SW1 Cherry_MX_RGB_WS2812, SW10 Cherry_MX_RGB_WS2812, SW11 Cherry_MX_RGB_WS2812, SW12 Cherry_MX_RGB_WS2812, SW13 Cherry_MX_RGB_WS2812, SW14 Cherry_MX_RGB_WS2812, SW15 Cherry_MX_RGB_WS2812, SW16 Cherry_MX_RGB_WS2812, SW19 Rotary_Encoder_Switch, SW2 Cherry_MX_RGB_WS2812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

Commit message: add resistor coming from LED pin
Parts:
- added R1: 470, Resistor_SMD:R_0805_2012Metric, B.Cu at (73.2, 37.8)
Connections:
- U1 pad 1: LED -> Net-(R1-Pad1)
Routing:
- net LED: track 59.9 -> 28.7 mm
- net Net-(R1-Pad1): track 0.00 -> 28.9 mm
Changed lines of the file:
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@@
     (thickness 1.6)
     (drawings 16)
-    (tracks 627)
+    (tracks 629)
     (zones 0)
-    (modules 61)
-    (nets 64)
+    (modules 62)
+    (nets 65)
   )
   (page A4)
@@
   (net 62 "Net-(D21-Pad4)")
   (net 63 "Net-(D22-Pad4)")
+  (net 64 "Net-(R1-Pad1)")
   (net_class Default "This is the default net class."
     (clearance 0.2)
@@
     (add_net "Net-(D8-Pad2)")
     (add_net "Net-(D9-Pad2)")
+    (add_net "Net-(R1-Pad1)")
     (add_net "Net-(SW1-Pad2)")
     (add_net "Net-(SW10-Pad2)")
@@
     (add_net VCC)
   )
+  (module Resistor_SMD:R_0805_2012Metric (layer B.Cu)
+    (at 73.152 37.846 270)
+    (descr "Resistor SMD 0805 (2012 Metric), square (rectangular) end terminal, IPC_7351 nominal, (Body size source: https://docs.google.com/spreadsheets/d/1BsfQQcO9C6DZCsRaXUlFlo91Tg2WpOkGARC1WS5S8t0/edit?usp=sharing), generated with kicad-footprint-generator")
+    (tags resistor)
+    (attr smd)
+    (fp_text reference R1 (at 0 1.65 90) (layer B.SilkS)
+      (effects (font (size 1 1) (thickness 0.15)) (justify mirror))
+    )
+    (fp_text value 470 (at 0 -1.65 90) (layer B.Fab)
+      (effects (font (size 1 1) (thickness 0.15)) (justify mirror))
+    )
+    (fp_text user %R (at 0 0 90) (layer B.Fab)
+      (effects (font (size 0.5 0.5) (thickness 0.08)) (justify mirror))
+    )
+    (fp_line (start -1 -0.6) (end -1 0.6) (layer B.Fab) (width 0.1))
+    (fp_line (start -1 0.6) (end 1 0.6) (layer B.Fab) (width 0.1))
+    (fp_line (start 1 0.6) (end 1 -0.6) (layer B.Fab) (width 0.1))
+    (fp_line (start 1 -0.6) (end -1 -0.6) (layer B.Fab) (width 0.1))
+    (fp_line (start -0.258578 0.71) (end 0.258578 0.71) (layer B.SilkS) (width 0.12))
+    (fp_line (start -0.258578 -0.71) (end 0.258578 -0.71) (layer B.SilkS) (width 0.12))
+    (fp_line (start -1.68 -0.95) (end -1.68 0.95) (layer B.CrtYd) (width 0.05))
+    (fp_line (start -1.68 0.95) (end 1.68 0.95) (layer B.CrtYd) (width 0.05))
+    (fp_line (start 1.68 0.95) (end 1.68 -0.95) (layer B.CrtYd) (width 0.05))
+    (fp_line (start 1.68 -0.95) (end -1.68 -0.95) (layer B.CrtYd) (width 0.05))
+    (pad 2 smd roundrect (at 0.9375 0 270) (size 0.975 1.4) (layers B.Cu B.Paste B.Mask) (roundrect_rratio 0.25)
+      (net 30 LED))
+    (pad 1 smd roundrect (at -0.9375 0 270) (size 0.975 1.4) (layers B.Cu B.Paste B.Mask) (roundrect_rratio 0.25)
+      (net 64 "Net-(R1-Pad1)"))
+    (model ${KISYS3DMOD}/Resistor_SMD.3dshapes/R_0805_2012Metric.wrl
+      (at (xyz 0 0 0))
+      (scale (xyz 1 1 1))
+      (rotate (xyz 0 0 0))
+    )
+  )
   (module MX_Only:MXOnly-2U-Hotswap (layer F.Cu)
     (at 120.65 112.776 270)
@@
     (fp_arc (start 0 41.989375) (end -4.318 17.8435) (angle 20.278025) (layer B.SilkS) (width 0.2032))
     (pad 1 smd roundrect (at -8.89 12.7 180) (size 2.54 1.27) (layers B.Cu B.Paste B.Mask) (roundrect_rratio 0.5)
-      (net 30 LED) (solder_mask_margin 0.1016))
+      (net 64 "Net-(R1-Pad1)") (solder_mask_margin 0.1016))
     (pad 2 smd roundrect (at -8.89 10.16 180) (size 2.54 1.27) (layers B.Cu B.Paste B.Mask) (roundrect_rratio 0.5)
       (net 48 "Net-(U1-Pad2)") (solder_mask_margin 0.1016))
@@
   (segment (start 71.12 88.138) (end 71.12 76.962) (width 0.254) (layer F.Cu) (net 29))
   (segment (start 71.12 76.962) (end 60.96 76.962) (width 0.254) (layer F.Cu) (net 29))
-  (via (at 73.152 36.322) (size 0.8) (drill 0.4) (layers F.Cu B.Cu) (net 30))
   (via (at 73.152 60.452) (size 0.8) (drill 0.4) (layers F.Cu B.Cu) (net 30))
-  (segment (start 73.152 36.322) (end 73.152 60.452) (width 0.254) (layer F.Cu) (net 30))
   (segment (start 66.1455 60.452) (end 66.1 60.4975) (width 0.254) (layer B.Cu) (net 30))
   (segment (start 73.152 60.452) (end 66.1455 60.452) (width 0.254) (layer B.Cu) (net 30))
-  (segment (start 73.152 36.322) (end 99.822 36.322) (width 0.254) (layer B.Cu) (net 30))
-  (segment (start 99.822 37.592) (end 100.33 38.1) (width 0.254) (layer B.Cu) (net 30))
-  (segment (start 99.822 36.322) (end 99.822 37.592) (width 0.254) (layer B.Cu) (net 30))
+  (via (at 73.152 41.402) (size 0.8) (drill 0.4) (layers F.Cu B.Cu) (net 30))
+  (segment (start 73.152 38.7835) (end 73.152 41.402) (width 0.254) (layer B.Cu) (net 30))
+  (segment (start 73.152 41.402) (end 73.152 60.452) (width 0.254) (layer F.Cu) (net 30))
   (via (at 60.96 91.44) (size 0.8) (drill 0.4) (layers F.Cu B.Cu) (net 31))
   (segment (start 60.9 91.38) (end 60.96 91.44) (width 0.254) (layer B.Cu) (net 31))
@@
   (segment (start 123.262 155.194) (end 123.25 155.206) (width 0.254) (layer B.Cu) (net 63))
   (segment (start 125.984 155.194) (end 123.262 155.194) (width 0.254) (layer B.Cu) (net 63))
+  (segment (start 99.822 36.322) (end 73.7385 36.322) (width 0.254) (layer B.Cu) (net 64))
+  (segment (start 73.7385 36.322) (end 73.152 36.9085) (width 0.254) (layer B.Cu) (net 64))
+  (segment (start 100.33 38.1) (end 99.822 37.592) (width 0.254) (layer B.Cu) (net 64))
+  (segment (start 99.822 37.592) (end 99.822 36.322) (width 0.254) (layer B.Cu) (net 64))
 )
