File: KiCad/Numpadulator.kicad_pcb (KiCad board)
At the start: 2 copper layers, 82.6 x 138.4 mm, 62 parts, among them SW1 Cherry_MX_RGB_WS2812, SW10 Cherry_MX_RGB_WS2812, SW11 Cherry_MX_RGB_WS2812, SW12 Cherry_MX_RGB_WS2812, SW13 Cherry_MX_RGB_WS2812, SW14 Cherry_MX_RGB_WS2812, SW15 Cherry_MX_RGB_WS2812, SW16 Cherry_MX_RGB_WS2812, SW19 Rotary_Encoder_Switch, SW2 Cherry_MX_RGB_WS2812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

Commit message: forgot to save
Parts:
- added C19: 0.1uF, Capacitor_SMD:C_0805_2012Metric, F.Cu at (168.1, 127.8)
- added C20: 0.1uF, Capacitor_SMD:C_0805_2012Metric, F.Cu at (168.1, 130.7)
- added C21: 0.1uF, Capacitor_SMD:C_0805_2012Metric, F.Cu at (172.6, 127.8)
- added C22: 0.1uF, Capacitor_SMD:C_0805_2012Metric, F.Cu at (172.6, 130.7)
- added C23: 0.1uF, Capacitor_SMD:C_0805_2012Metric, F.Cu at (177.0, 127.8)
- added C24: 0.1uF, Capacitor_SMD:C_0805_2012Metric, F.Cu at (177.0, 130.7)
- added D23: SK6812MINI, LED_SMD:LED_SK6812MINI_PLCC4_3.5x3.5mm_P1.75mm, F.Cu at (24.1, 71.1)
- added D24: SK6812MINI, LED_SMD:LED_SK6812MINI_PLCC4_3.5x3.5mm_P1.75mm, F.Cu at (24.1, 76.2)
- added D25: SK6812MINI, LED_SMD:LED_SK6812MINI_PLCC4_3.5x3.5mm_P1.75mm, F.Cu at (31.1, 71.1)
- added D26: SK6812MINI, LED_SMD:LED_SK6812MINI_PLCC4_3.5x3.5mm_P1.75mm, F.Cu at (31.1, 76.2)
- added D27: SK6812MINI, LED_SMD:LED_SK6812MINI_PLCC4_3.5x3.5mm_P1.75mm, F.Cu at (38.2, 71.1)
- added D28: SK6812MINI, LED_SMD:LED_SK6812MINI_PLCC4_3.5x3.5mm_P1.75mm, F.Cu at (38.2, 76.2)
Connections:
- D22 pad 2: Net-(D20-Pad4) -> Net-(D22-Pad2)
- SW1 pad 2: Net-(SW1-Pad2) -> Net-(D23-Pad3)
- SW2 pad 4: Net-(SW1-Pad2) -> Net-(D24-Pad1)
- SW3 pad 2: Net-(SW3-Pad2) -> Net-(D25-Pad3)
- SW8 pad 4: Net-(SW3-Pad2) -> Net-(D25-Pad1)

Commit message: PLACED EVERYTHING I THINK
Parts:
- C19, C20, C21, C22, C23, C24, D23, D24, D25, D26, D27, D28: moved to B.Cu
- moved C21 128.2 mm to (59.9, 66.5), turned to 90 degrees
- moved D28 119.3 mm to (120.7, 162.3), turned to 180 degrees
- moved C20 112.8 mm to (59.7, 161.8)
- moved C19 109.7 mm to (59.4, 113.3)
- moved D26 106.9 mm to (129.5, 117.9)
- moved D24 96.8 mm to (120.7, 68.3), turned to 180 degrees
- moved D27 91.2 mm to (54.9, 160.8)
- moved C22 84.8 mm to (116.8, 66.8), turned to 90 degrees
- moved C23 69.6 mm to (116.6, 162.3), turned to 270 degrees
- moved D25 47.7 mm to (54.9, 112.5)
- moved C24 47.3 mm to (130.6, 121.4), turned to 270 degrees
- moved D23 39.7 mm to (63.8, 68.3), turned to 180 degrees
Connections:
- D26 pad 1: Net-(D21-Pad2) -> Net-(D26-Pad1)
- SW4 pad 4: Net-(D21-Pad2) -> Net-(D26-Pad1)
Routing:
- net VCC: track 545.4 -> 675.5 mm, vias 7 -> 11
- net Net-(D24-Pad1): track 0.00 -> 91.8 mm, vias 0 -> 2
- net Net-(D26-Pad1): track 0.00 -> 80.3 mm, vias 0 -> 2
- net Net-(D22-Pad2): track 0.00 -> 69.9 mm, vias 0 -> 2
- net Net-(D23-Pad1): track 0.00 -> 56.5 mm
- net Net-(D21-Pad2): track 69.3 -> 16.1 mm, vias 2 -> 0
- net Net-(SW1-Pad2): track 41.7 -> 0.00 mm, vias 2 -> 0
- net Net-(D25-Pad1): track 0.00 -> 40.1 mm, vias 0 -> 2
- net Net-(SW3-Pad2): track 32.5 -> 0.00 mm, vias 2 -> 0
- net Net-(D28-Pad3): track 0.00 -> 27.1 mm, vias 0 -> 2
- net Net-(D20-Pad4): track 60.7 -> 39.5 mm
- net Net-(D23-Pad3): track 0.00 -> 13.1 mm
- net Net-(D25-Pad3): track 0.00 -> 5.39 mm

Commit message: made some GND SPACE
Routing:
- net Net-(D21-Pad4): track 40.0 -> 42.5 mm
Changed lines of the file:
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@@
     (thickness 1.6)
     (drawings 16)
-    (tracks 717)
+    (tracks 718)
     (zones 0)
     (modules 74)
@@
   (segment (start 107.636038 112.779538) (end 116.2685 121.412) (width 0.254) (layer F.Cu) (net 59))
   (segment (start 116.2685 121.412) (end 125.349 121.412) (width 0.254) (layer F.Cu) (net 59))
-  (via (at 125.222 117.094) (size 0.8) (drill 0.4) (layers F.Cu B.Cu) (net 59))
-  (segment (start 125.349 121.412) (end 125.349 117.221) (width 0.254) (layer F.Cu) (net 59))
-  (segment (start 125.349 117.221) (end 125.222 117.094) (width 0.254) (layer F.Cu) (net 59))
   (segment (start 123.262 117.094) (end 123.25 117.106) (width 0.254) (layer B.Cu) (net 59))
-  (segment (start 125.222 117.094) (end 123.262 117.094) (width 0.254) (layer B.Cu) (net 59))
+  (segment (start 125.349 121.412) (end 125.349 117.221) (width 0.254) (layer F.Cu) (net 59))
+  (via (at 123.444 115.316) (size 0.8) (drill 0.4) (layers F.Cu B.Cu) (net 59))
+  (segment (start 125.349 117.221) (end 123.444 115.316) (width 0.254) (layer F.Cu) (net 59))
+  (segment (start 123.444 116.912) (end 123.25 117.106) (width 0.254) (layer B.Cu) (net 59))
+  (segment (start 123.444 115.316) (end 123.444 116.912) (width 0.254) (layer B.Cu) (net 59))
   (via (at 99.06 148.59) (size 0.8) (drill 0.4) (layers F.Cu B.Cu) (net 60))
   (segment (start 99 148.53) (end 99.06 148.59) (width 0.254) (layer B.Cu) (net 60))

Commit message: now.. they should be placed right... maybe...
Routing:
- net VCC: track 675.5 -> 666.3 mm, vias 11 -> 13
- net ROTB: track 63.2 -> 64.3 mm, vias 2 -> 4
- net Net-(D21-Pad2): vias 0 -> 2

Commit message: jk for real this time lololol
Routing:
- net Net-(D20-Pad2): track 47.1 -> 46.0 mm
Changed lines of the file:
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@@
     (thickness 1.6)
     (drawings 16)
-    (tracks 734)
+    (tracks 735)
     (zones 0)
     (modules 74)
@@
   (segment (start 83.566 165.354) (end 86.36 165.354) (width 0.254) (layer B.Cu) (net 56))
   (segment (start 86.36 165.354) (end 89.154 168.148) (width 0.254) (layer B.Cu) (net 56))
-  (segment (start 107.188 168.148) (end 107.188 164.592) (width 0.254) (layer B.Cu) (net 56))
-  (segment (start 107.188 164.592) (end 104.648 164.592) (width 0.254) (layer B.Cu) (net 56))
   (segment (start 89.154 168.148) (end 89.154 168.148) (width 0.254) (layer B.Cu) (net 56))
   (via (at 89.154 168.148) (size 0.8) (drill 0.4) (layers F.Cu B.Cu) (net 56))
-  (via (at 107.188 168.148) (size 0.8) (drill 0.4) (layers F.Cu B.Cu) (net 56))
-  (segment (start 89.154 168.148) (end 107.188 168.148) (width 0.254) (layer F.Cu) (net 56))
+  (segment (start 89.154 168.148) (end 106.426 168.148) (width 0.254) (layer F.Cu) (net 56))
+  (via (at 106.426 164.592) (size 0.8) (drill 0.4) (layers F.Cu B.Cu) (net 56))
+  (segment (start 106.426 168.148) (end 106.426 164.592) (width 0.254) (layer F.Cu) (net 56))
+  (segment (start 104.2455 164.592) (end 104.2 164.6375) (width 0.254) (layer B.Cu) (net 56))
+  (segment (start 106.426 164.592) (end 104.2455 164.592) (width 0.254) (layer B.Cu) (net 56))
   (segment (start 106.68 150.622) (end 79.756 150.622) (width 0.254) (layer F.Cu) (net 69))
   (via (at 79.756 164.338) (size 0.8) (drill 0.4) (layers F.Cu B.Cu) (net 57))

Commit message: 10,000th times the charm!
Routing:
- net ROW5: track 232.2 -> 234.2 mm
Changed lines of the file:
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@@
     (thickness 1.6)
     (drawings 16)
-    (tracks 735)
+    (tracks 736)
     (zones 0)
     (modules 74)
@@
   (via (at 132.588 165.354) (size 0.8) (drill 0.4) (layers F.Cu B.Cu) (net 14))
   (segment (start 132.588 73.152) (end 132.588 165.354) (width 0.254) (layer F.Cu) (net 14))
-  (segment (start 108.838 165.354) (end 108.712 165.48) (width 0.254) (layer B.Cu) (net 14))
-  (segment (start 132.588 165.354) (end 108.838 165.354) (width 0.254) (layer B.Cu) (net 14))
   (segment (start 106.600501 162.664501) (end 100.434501 162.664501) (width 0.254) (layer B.Cu) (net 14))
   (segment (start 108.712 165.48) (end 108.712 164.776) (width 0.254) (layer B.Cu) (net 14))
@@
   (segment (start 99.7575 161.9875) (end 80.9625 161.9875) (width 0.254) (layer B.Cu) (net 14))
   (segment (start 100.434501 162.664501) (end 99.7575 161.9875) (width 0.254) (layer B.Cu) (net 14))
+  (segment (start 111.126 167.894) (end 108.712 165.48) (width 0.254) (layer B.Cu) (net 14))
+  (segment (start 132.588 165.354) (end 130.048 167.894) (width 0.254) (layer B.Cu) (net 14))
+  (segment (start 130.048 167.894) (end 111.126 167.894) (width 0.254) (layer B.Cu) (net 14))
   (segment (start 88.565 80.565) (end 90.4875 82.4875) (width 0.254) (layer B.Cu) (net 15))
   (segment (start 88.565 79.0575) (end 88.565 80.565) (width 0.254) (layer B.Cu) (net 15))

Commit message: I crave... something
Routing:
- net ROW5: track 234.2 -> 237.2 mm, vias 4 -> 5
Changed lines of the file:
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@@
     (thickness 1.6)
     (drawings 16)
-    (tracks 736)
+    (tracks 738)
     (zones 0)
     (modules 74)
@@
   (segment (start 99.7575 161.9875) (end 80.9625 161.9875) (width 0.254) (layer B.Cu) (net 14))
   (segment (start 100.434501 162.664501) (end 99.7575 161.9875) (width 0.254) (layer B.Cu) (net 14))
-  (segment (start 111.126 167.894) (end 108.712 165.48) (width 0.254) (layer B.Cu) (net 14))
-  (segment (start 132.588 165.354) (end 130.048 167.894) (width 0.254) (layer B.Cu) (net 14))
-  (segment (start 130.048 167.894) (end 111.126 167.894) (width 0.254) (layer B.Cu) (net 14))
+  (via (at 108.712 166.624) (size 0.8) (drill 0.4) (layers F.Cu B.Cu) (net 14))
+  (segment (start 108.712 165.48) (end 108.712 166.624) (width 0.254) (layer B.Cu) (net 14))
+  (segment (start 127.288999 170.653001) (end 132.588 165.354) (width 0.254) (layer F.Cu) (net 14))
+  (segment (start 112.741001 170.653001) (end 127.288999 170.653001) (width 0.254) (layer F.Cu) (net 14))
+  (segment (start 108.712 166.624) (end 112.741001 170.653001) (width 0.254) (layer F.Cu) (net 14))
   (segment (start 88.565 80.565) (end 90.4875 82.4875) (width 0.254) (layer B.Cu) (net 15))
   (segment (start 88.565 79.0575) (end 88.565 80.565) (width 0.254) (layer B.Cu) (net 15))

Commit message: lolol
Routing:
- net ROW5: vias 5 -> 4
Changed lines of the file:
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@@
     (thickness 1.6)
     (drawings 16)
-    (tracks 738)
+    (tracks 737)
     (zones 0)
     (modules 74)
@@
   (via (at 132.588 73.152) (size 0.8) (drill 0.4) (layers F.Cu B.Cu) (net 14))
   (segment (start 66.548 73.152) (end 132.588 73.152) (width 0.254) (layer B.Cu) (net 14))
-  (via (at 132.588 165.354) (size 0.8) (drill 0.4) (layers F.Cu B.Cu) (net 14))
   (segment (start 132.588 73.152) (end 132.588 165.354) (width 0.254) (layer F.Cu) (net 14))
   (segment (start 106.600501 162.664501) (end 100.434501 162.664501) (width 0.254) (layer B.Cu) (net 14))
